Commit message: update slam config v2

File: description/robot.urdf.xacro (robot description, xacro)
@@ -1,6 +1,5 @@
 <?xml version="1.0"?>
-<robot xmlns:xacro="http://www.ros.org/wiki/xacro"  name="robot">
-    <!-- Example link -->
-    <xacro:include filename="robot_core.xacro"/>
-    <xacro:include filename="gazebo_control.xacro"/>
+<robot xmlns:xacro="http://www.ros.org/wiki/xacro" name="hoainam_robot">
+  <xacro:include filename="robot_core.xacro"/>
+  <xacro:include filename="lidar.xacro"/>
 </robot>

File: description/robot_core.xacro (robot description, xacro)
@@ -1,125 +1,136 @@
 <?xml version="1.0"?>
-<robot xmlns:xacro="http://www.ros.org/wiki/xacro"  >
-    <xacro:include filename="inertial_macros.xacro"/>
-    <material name="white">
-        <color rgba="1 1 1 1" />
-    </material>
-    <material name="orange">
-        <color rgba="1 0.3 0.1 1" />
-    </material>
-    <material name="blue">
-        <color rgba="0.2 0.2 1 1" />
-    </material>
-    <material name="black">
-        <color rgba="0 0 0 1" />
-    </material>
-        <!-- BASE LINK-->
-    <link name="base_link">
-    </link>
-        <!-- CHASSIS LINK-->
-    <joint name="chassis_joint" type="fixed">
-        <parent link="base_link"/>
-        <child link="chassis"/>
-        <origin xyz="-0.13 0 0"/>
-    </joint>
-    <link name="chassis">
-        <visual>
-            <origin xyz="0.5 0 0.3"/>
-            <geometry>
-                <box size="1 0.6 0.6"/>
-            </geometry>
-            <material name="white"/>
-        </visual>
-        <collision>
-            <origin xyz="0.5 0 0.3"/>
-            <geometry>
-                <box size="1 0.6 0.6"/>
-            </geometry>
-        </collision>
-        <xacro:inertial_box mass="60" x="1" y="0.6" z="0.6">
-            <origin xyz="0.5 0 0.3" rpy="0 0 0"/>
-        </xacro:inertial_box>
-    </link>
-    <gazebo reference="chassis">
-        <material>Gazebo/White</material>
-    </gazebo>
-        <!-- LEFT WHEEL LINK -->
-    <joint name="left_wheel_joint" type="continuous">
-        <parent link="base_link"/>
-        <child link = "left_wheel"/>
-        <origin xyz="0 0.21 0" rpy="-${pi/2} 0 0"/>
-        <axis xyz="0 0 1"/>
-    </joint>
-    <link name="left_wheel">
-        <visual>
-            <geometry>
-                <cylinder radius="0.0605" length="0.03"/>
-            </geometry>
-            <material name="blue"/>
-        </visual>
-        <collision>
-            <geometry>
-                <cylinder radius="0.0605" length="0.03"/>
-            </geometry>
-        </collision>
-        <xacro:inertial_cylinder mass="0.5" length="0.03" radius="0.0605">
-            <origin xyz="0 0 0" rpy="0 0 0"/>
-        </xacro:inertial_cylinder>
-    </link>
-    <gazebo reference="left_wheel">
-        <material>Gazebo/Blue</material>
-    </gazebo>
-        <!-- RIGHT WHEEL LINK -->
-    <joint name="right_wheel_joint" type="continuous">
-        <parent link="base_link"/>
-        <child link = "right_wheel"/>
-        <origin xyz="0 -0.21 0" rpy="${pi/2} 0 0"/>
-        <axis xyz="0 0 -1"/>
-    </joint>
-    <link name="right_wheel">
-        <visual>
-            <geometry>
-                <cylinder radius="0.0625" length="0.03"/>
-            </geometry>
-            <material name="blue"/>
-        </visual>
-        <collision>
-            <geometry>
-                <cylinder radius="0.0625" length="0.03"/>
-            </geometry>
-        </collision>
-        <xacro:inertial_cylinder mass="0.5" length="0.03" radius="0.0625">
-            <origin xyz="0 0 0" rpy="0 0 0"/>
-        </xacro:inertial_cylinder>
-    </link>
-    <gazebo reference="right_wheel">
-        <material>Gazebo/Blue</material>
-    </gazebo>
-        <!-- CASTER WHEEL LINK -->
-    <joint name="caster_wheel_joint" type="fixed">
-        <parent link="chassis"/>
-        <child link="caster_wheel"/>
-        <origin xyz="0.85 0 0"/>
-    </joint>
-    <link name="caster_wheel">
-        <visual>
-            <geometry>
-                <sphere radius="0.0625"/>
-            </geometry>
-            <material name="black"/>
-        </visual>
-        <collision>
-            <geometry>
-                <sphere radius="0.0625"/>
-            </geometry>
-        </collision>
-        <xacro:inertial_sphere mass="0.1" radius="0.0625">
-            <origin xyz="0 0 0" rpy="0 0 0"/>
-        </xacro:inertial_sphere>
-    </link>
-    <gazebo reference="caster_wheel">
-        <material>Gazebo/Black</material>
-        <mu1 value="0.001"/>
-        <mu2 value="0.001"/>
-    </gazebo>
+<robot xmlns:xacro="http://www.ros.org/wiki/xacro" >
+<xacro:include filename="inertial_macros.xacro"/>
+<material name="white">
+<color rgba="1 1 1 1" />
+</material>
+<material name="orange">
+<color rgba="1 0.3 0.1 1" />
+</material>
+<material name="blue">
+<color rgba="0.2 0.2 1 1" />
+</material>
+<material name="black">
+<color rgba="0 0 0 1" />
+</material>
+<material name="red">
+<color rgba="1 0 0 1" />
+</material>
+<!-- BASE LINK-->
+<link name="base_link">
+</link>
+<!-- BASE FOOTPRINT LINK -->
+<joint name="base_footprint_joint" type="fixed">
+<parent link="base_footprint"/>
+<child link="base_link"/>
+<origin xyz="0 0 0" rpy="0 0 0"/>
+</joint>
+<link name="base_footprint">
+</link>
+<!-- CHASSIS LINK-->
+<joint name="chassis_joint" type="fixed">
+<parent link="base_link"/>
+<child link="chassis"/>
+<origin xyz="-0.13 0 0"/>
+</joint>
+<link name="chassis">
+<visual>
+<origin xyz="0.5 0 0.3"/>
+<geometry>
+<box size="1 0.6 0.6"/>
+</geometry>
+<material name="orange"/>
+</visual>
+<collision>
+<origin xyz="0.5 0 0.3"/>
+<geometry>
+<box size="1 0.6 0.6"/>
+</geometry>
+</collision>
+<xacro:inertial_box mass="60" x="1" y="0.6" z="0.6">
+<origin xyz="0.5 0 0.3" rpy="0 0 0"/>
+</xacro:inertial_box>
+</link>
+<gazebo reference="chassis">
+<material>Gazebo/Orange</material>
+</gazebo>
+<!-- LEFT WHEEL LINK -->
+<joint name="left_wheel_joint" type="continuous">
+<parent link="base_link"/>
+<child link = "left_wheel"/>
+<origin xyz="0 0.21 0" rpy="-${pi/2} 0 0"/>
+<axis xyz="0 0 1"/>
+</joint>
+<link name="left_wheel">
+<visual>
+<geometry>
+<cylinder radius="0.0605" length="0.03"/>
+</geometry>
+<material name="blue"/>
+</visual>
+<collision>
+<geometry>
+<cylinder radius="0.0605" length="0.03"/>
+</geometry>
+</collision>
+<xacro:inertial_cylinder mass="0.5" length="0.03" radius="0.0605">
+<origin xyz="0 0 0" rpy="0 0 0"/>
+</xacro:inertial_cylinder>
+</link>
+<gazebo reference="left_wheel">
+<material>Gazebo/Blue</material>
+</gazebo>
+<!-- RIGHT WHEEL LINK -->
+<joint name="right_wheel_joint" type="continuous">
+<parent link="base_link"/>
+<child link = "right_wheel"/>
+<origin xyz="0 -0.21 0" rpy="${pi/2} 0 0"/>
+<axis xyz="0 0 -1"/>
+</joint>
+<link name="right_wheel">
+<visual>
+<geometry>
+<cylinder radius="0.0625" length="0.03"/>
+</geometry>
+<material name="blue"/>
+</visual>
+<collision>
+<geometry>
+<cylinder radius="0.0625" length="0.03"/>
+</geometry>
+</collision>
+<xacro:inertial_cylinder mass="0.5" length="0.03" radius="0.0625">
+<origin xyz="0 0 0" rpy="0 0 0"/>
+</xacro:inertial_cylinder>
+</link>
+<gazebo reference="right_wheel">
+<material>Gazebo/Blue</material>
+</gazebo>
+<!-- CASTER WHEEL LINK -->
+<joint name="caster_wheel_joint" type="fixed">
+<parent link="chassis"/>
+<child link="caster_wheel"/>
+<origin xyz="0.85 0 0"/>
+</joint>
+<link name="caster_wheel">
+<visual>
+<geometry>
+<sphere radius="0.0625"/>
+</geometry>
+<material name="black"/>
+</visual>
+<collision>
+<geometry>
+<sphere radius="0.0625"/>
+</geometry>
+</collision>
+<xacro:inertial_sphere mass="0.1" radius="0.0625">
+<origin xyz="0 0 0" rpy="0 0 0"/>
+</xacro:inertial_sphere>
+</link>
+<gazebo reference="caster_wheel">
+<material>Gazebo/Black</material>
+<mu1 value="0.001"/>
+<mu2 value="0.001"/>
+</gazebo>
 </robot>
