Commit message: update rviz config and robot model

File: description/robot_core.xacro (robot description, xacro)
@@ -21,22 +21,22 @@
         <parent link="base_link"/>
         <child link="chassis"/>
-        <origin xyz="-0.1 0 0"/>
+        <origin xyz="-0.13 0 0"/>
     </joint>
     <link name="chassis">
         <visual>
-            <origin xyz="0.15 0 0.075"/>
+            <origin xyz="0.5 0 0.3"/>
             <geometry>
-                <box size="0.3 0.3 0.15"/>
+                <box size="1 0.6 0.6"/>
             </geometry>
             <material name="white"/>
         </visual>
         <collision>
-            <origin xyz="0.15 0 0.075"/>
+            <origin xyz="0.5 0 0.3"/>
             <geometry>
-                <box size="0.3 0.3 0.15"/>
+                <box size="1 0.6 0.6"/>
             </geometry>
         </collision>
-        <xacro:inertial_box mass="0.5" x="0.3" y="0.3" z="0.15">
-            <origin xyz="0.15 0 0.075" rpy="0 0 0"/>
+        <xacro:inertial_box mass="60" x="1" y="0.6" z="0.6">
+            <origin xyz="0.5 0 0.3" rpy="0 0 0"/>
         </xacro:inertial_box>
     </link>
@@ -45,5 +45,5 @@
         <parent link="base_link"/>
         <child link = "left_wheel"/>
-        <origin xyz="0 0.175 0" rpy="-${pi/2} 0 0"/>
+        <origin xyz="0 0.21 0" rpy="-${pi/2} 0 0"/>
         <axis xyz="0 0 1"/>
     </joint>
@@ -51,5 +51,5 @@
         <visual>
             <geometry>
-                <cylinder radius="0.05" length="0.04"/>
+                <cylinder radius="0.0605" length="0.03"/>
             </geometry>
             <material name="blue"/>
@@ -57,8 +57,8 @@
         <collision>
             <geometry>
-                <cylinder radius="0.05" length="0.04"/>
+                <cylinder radius="0.0605" length="0.03"/>
             </geometry>
         </collision>
-        <xacro:inertial_cylinder mass="0.1" length="0.04" radius="0.05">
+        <xacro:inertial_cylinder mass="0.5" length="0.03" radius="0.0605">
             <origin xyz="0 0 0" rpy="0 0 0"/>
         </xacro:inertial_cylinder>
@@ -68,5 +68,5 @@
         <parent link="base_link"/>
         <child link = "right_wheel"/>
-        <origin xyz="0 -0.175 0" rpy="${pi/2} 0 0"/>
+        <origin xyz="0 -0.21 0" rpy="${pi/2} 0 0"/>
         <axis xyz="0 0 -1"/>
     </joint>
@@ -74,5 +74,5 @@
         <visual>
             <geometry>
-                <cylinder radius="0.05" length="0.04"/>
+                <cylinder radius="0.0605" length="0.03"/>
             </geometry>
             <material name="blue"/>
@@ -80,8 +80,8 @@
         <collision>
             <geometry>
-                <cylinder radius="0.05" length="0.04"/>
+                <cylinder radius="0.0605" length="0.03"/>
             </geometry>
         </collision>
-        <xacro:inertial_cylinder mass="0.1" length="0.04" radius="0.05">
+        <xacro:inertial_cylinder mass="0.5" length="0.03" radius="0.0605">
             <origin xyz="0 0 0" rpy="0 0 0"/>
         </xacro:inertial_cylinder>
@@ -91,10 +91,10 @@
         <parent link="chassis"/>
         <child link="caster_wheel"/>
-        <origin xyz="0.24 0 0"/>
+        <origin xyz="0.85 0 0"/>
     </joint>
     <link name="caster_wheel">
         <visual>
             <geometry>
-                <sphere radius="0.05"/>
+                <sphere radius="0.0605"/>
             </geometry>
             <material name="black"/>
@@ -102,8 +102,8 @@
         <collision>
             <geometry>
-                <sphere radius="0.05"/>
+                <sphere radius="0.0605"/>
             </geometry>
         </collision>
-        <xacro:inertial_sphere mass="0.1" radius="0.05">
+        <xacro:inertial_sphere mass="0.1" radius="0.0605">
             <origin xyz="0 0 0" rpy="0 0 0"/>
         </xacro:inertial_sphere>

Commit message: update launch file

File: description/robot_core.xacro (robot description, xacro)
@@ -41,4 +41,7 @@
         </xacro:inertial_box>
     </link>
+    <gazebo reference="chassis">
+        <material>Gazebo/White</material>
+    </gazebo>
         <!-- LEFT WHEEL LINK -->
     <joint name="left_wheel_joint" type="continuous">
@@ -64,4 +67,7 @@
         </xacro:inertial_cylinder>
     </link>
+    <gazebo reference="left_wheel">
+        <material>Gazebo/Blue</material>
+    </gazebo>
         <!-- RIGHT WHEEL LINK -->
     <joint name="right_wheel_joint" type="continuous">
@@ -74,5 +80,5 @@
         <visual>
             <geometry>
-                <cylinder radius="0.0605" length="0.03"/>
+                <cylinder radius="0.0625" length="0.03"/>
             </geometry>
             <material name="blue"/>
@@ -80,11 +86,14 @@
         <collision>
             <geometry>
-                <cylinder radius="0.0605" length="0.03"/>
+                <cylinder radius="0.0625" length="0.03"/>
             </geometry>
         </collision>
-        <xacro:inertial_cylinder mass="0.5" length="0.03" radius="0.0605">
+        <xacro:inertial_cylinder mass="0.5" length="0.03" radius="0.0625">
             <origin xyz="0 0 0" rpy="0 0 0"/>
         </xacro:inertial_cylinder>
     </link>
+    <gazebo reference="right_wheel">
+        <material>Gazebo/Blue</material>
+    </gazebo>
         <!-- CASTER WHEEL LINK -->
     <joint name="caster_wheel_joint" type="fixed">
@@ -96,5 +105,5 @@
         <visual>
             <geometry>
-                <sphere radius="0.0605"/>
+                <sphere radius="0.0625"/>
             </geometry>
             <material name="black"/>
@@ -102,10 +111,15 @@
         <collision>
             <geometry>
-                <sphere radius="0.0605"/>
+                <sphere radius="0.0625"/>
             </geometry>
         </collision>
-        <xacro:inertial_sphere mass="0.1" radius="0.0605">
+        <xacro:inertial_sphere mass="0.1" radius="0.0625">
             <origin xyz="0 0 0" rpy="0 0 0"/>
         </xacro:inertial_sphere>
     </link>
+    <gazebo reference="caster_wheel">
+        <material>Gazebo/Black</material>
+        <mu1 value="0.001"/>
+        <mu2 value="0.001"/>
+    </gazebo>
 </robot>

Commit message: update launch + slam config for RF2O + fix urdf

File: description/robot_core.xacro (robot description, xacro)
@@ -3,17 +3,17 @@
 <xacro:include filename="inertial_macros.xacro"/>
 <material name="white">
-<color rgba="1 1 1 1" />
+    <color rgba="1 1 1 1" />
 </material>
 <material name="orange">
-<color rgba="1 0.3 0.1 1" />
+    <color rgba="1 0.3 0.1 1" />
 </material>
 <material name="blue">
-<color rgba="0.2 0.2 1 1" />
+    <color rgba="0.2 0.2 1 1" />
 </material>
 <material name="black">
-<color rgba="0 0 0 1" />
+    <color rgba="0 0 0 1" />
 </material>
 <material name="red">
-<color rgba="1 0 0 1" />
+    <color rgba="1 0 0 1" />
 </material>
 <!-- BASE LINK-->
@@ -22,7 +22,7 @@
 <!-- BASE FOOTPRINT LINK -->
 <joint name="base_footprint_joint" type="fixed">
-<parent link="base_footprint"/>
-<child link="base_link"/>
-<origin xyz="0 0 0" rpy="0 0 0"/>
+    <parent link="base_footprint"/>
+    <child link="base_link"/>
+    <origin xyz="0 0 0" rpy="0 0 0"/>
 </joint>
 <link name="base_footprint">
@@ -30,25 +30,25 @@
 <!-- CHASSIS LINK-->
 <joint name="chassis_joint" type="fixed">
-<parent link="base_link"/>
-<child link="chassis"/>
-<origin xyz="-0.13 0 0"/>
+    <parent link="base_link"/>
+    <child link="chassis"/>
+    <origin xyz="-0.13 0 0"/>
 </joint>
 <link name="chassis">
-<visual>
-<origin xyz="0.5 0 0.3"/>
-<geometry>
-<box size="1 0.6 0.6"/>
-</geometry>
-<material name="orange"/>
-</visual>
-<collision>
-<origin xyz="0.5 0 0.3"/>
-<geometry>
-<box size="1 0.6 0.6"/>
-</geometry>
-</collision>
-<xacro:inertial_box mass="60" x="1" y="0.6" z="0.6">
-<origin xyz="0.5 0 0.3" rpy="0 0 0"/>
-</xacro:inertial_box>
+    <visual>
+        <origin xyz="0.5 0 0.3"/>
+        <geometry>
+            <box size="1 0.6 0.6"/>
+        </geometry>
+        <material name="orange"/>
+    </visual>
+    <collision>
+        <origin xyz="0.5 0 0.3"/>
+        <geometry>
+        <box size="1 0.6 0.6"/>
+        </geometry>
+    </collision>
+    <xacro:inertial_box mass="60" x="1" y="0.6" z="0.6">
+    <origin xyz="0.5 0 0.3" rpy="0 0 0"/>
+    </xacro:inertial_box>
 </link>
 <gazebo reference="chassis">
@@ -65,5 +65,5 @@
 <visual>
 <geometry>
-<cylinder radius="0.0605" length="0.03"/>
+<cylinder radius="0.0625" length="0.03"/>
 </geometry>
 <material name="blue"/>
@@ -71,8 +71,8 @@
 <collision>
 <geometry>
-<cylinder radius="0.0605" length="0.03"/>
+<cylinder radius="0.0625" length="0.03"/>
 </geometry>
 </collision>
-<xacro:inertial_cylinder mass="0.5" length="0.03" radius="0.0605">
+<xacro:inertial_cylinder mass="0.5" length="0.03" radius="0.0625">
 <origin xyz="0 0 0" rpy="0 0 0"/>
 </xacro:inertial_cylinder>
